File: Cosmic Pi V2.sch (EAGLE design)
At the start: 191 parts, among them IC1 AD8039, IC2 AD8039, IC3 LP2985IM5-3.1, IC4 LM555D, IC5 LM555D, IC6 LM555D, IC7 74AUC1G00DBV, IC8 74AUC1G00DBV, IC9 74AUC1G00DBV, J1 U.FL-R-SMT-1(10), J10 2p-2.54, J11 2p-2.54, J2 U.FL-R-SMT-1(10), J3 4p-2.54, J4 4p-2.54, J5 5-1814400-1, J6 2p-2.54, J7 2p-2.54, J8 2p-2.54, J9 2p-2.54, Q1 BSS123, Q2 BSS123, U1 L76-M33, U2 LSM303D, U5 MAX1932, U6 MAX1932, X1 22-23-2041, X2 22-23-2041, X3 22-23-2021, X4 22-23-2051

Commit message: Work in progress
Added DACs.
Tidied Sheet 1 - Analogue.
Started Adding STM32's (one of two).
To do: 1 - 1mm2 SiPM Footprint
2 - Finish STM32s (2)
3- Power regulator + jack
Parts:
- removed DUE1: DUE(NORMAL), DUElib130425:DUE(NORMAL)
- removed J3, J4: 4p-2.54, Seeed-Connector:DIP-BLACK-FEMALE-HEADER-VERT(4P-2.54)
- removed J6: 2p-2.54, Seeed-Connector:DIP-BLACK-MALE-HEADER-VERT(2P-2.54)
- removed X1: 22-23-2041, con-molex:22-23-2041
- removed X3: 22-23-2021, con-molex:22-23-2021
- added C65, C66: 100n, resistor:C-EUC0603
- added C67, C68: 10u, resistor:C-EUC0603
- added C69, C70: 20p, rcl:C-EUC0603
- added C71: 4.7u, resistor:C-EUC0603
- added U$10: 310010495_STM32F401RET6, Seeed-OPL-2017-01-IC-Akita:310010495_STM32F401RET6
- added U3, U4: MCP4725, SparkFun-IC-Conversion:MCP4725SOT-23
- X2: value 22-23-2041 -> 306010282_XTAL_8MHZ-HC49US; device con-molex:22-23-2041 -> Seeed-OPL-2017-01-Crystal-Akita:306010282_XTAL_8MHZ-HC49US
Connections:
- removed net AMP2B: DUE1.A7, IC$3.INB+, J3.P$1
- removed net DREF1: DUE1.A1
- removed net DREF2: DUE1.A2
- removed net EXTGPSFIX: DUE1.4
- removed net HTU3V: DUE1.9
- removed net IMU3V: DUE1.8
- removed net N$12: R4.2, R5.2, X3-2.S
- removed net PA0: DUE1.A9
- removed net PA1: DUE1.A10
- removed net PA2: DUE1.A11
- removed net TEMPA: J6.1
- removed net TEMPB: J6.2
- new net +5FV: C7.1, IC3.ON/OFF, IC3.VIN, L1.3, R6.1
- new net AGND: C11.2, C14.2, C15.2, C19.2, C2.2, C20.2, C21.2, C22.2, C24.2, C25.2, C3.2, C6.-, C7.2, C8.2, IC1P.V-, IC2P.V-, IC3.GND, L1.2, LED1.C, LED2.C, R32.1
- new net N$21: U$10.VSSA
- new net N$49: U$10.VSS1
- new net N$51: U$10.VSS2
- new net N$62: C71.2, U$10.VCAP
- new net TEMP1: R4.1, R5.1
- new net TEMP2: R4.2, R5.2
- net !RESET: no longer DUE1.RESET
- net +3V3: now also U$10.VDD, U$10.VDD3, U$10.VDDA; no longer DUE1.3V3
- net +5V: no longer C7.1, DUE1.5V, IC3.ON/OFF, IC3.VIN, J4.P$1, L1.3, R6.1
- net ACCELINT1: no longer DUE1.10
- net ACCELINT2: no longer DUE1.13
- net ACCELINT3: no longer DUE1.SDA1
- net ACCELSA0: no longer DUE1.6
- net ACCELSA1: no longer DUE1.7
- net AMP2A: no longer DUE1.A6, J3.P$3
- net GND: now also C65.1, C66.1, C67.1, C68.1, C69.1, C71.1, L1.1, U$10.VSS, U$10.VSS3, U3.VSS, U4.AO, U4.VSS; no longer C11.2, C14.2, C15.2, C19.2, C2.2, C20.2, C21.2, C22.2, C24.2, C25.2, C3.2, C6.-, C7.2, C8.2, DUE1.GND1, DUE1.GND_1, DUE1.GND_2, DUE1.GND_A, DUE1.GND_B, IC1P.V-, IC2P.V-, IC3.GND, J3.P$2, J4.P$2, L1.2, LED1.C, LED2.C, R32.1, X1-3.S
- net GPSPPS: no longer DUE1.2
- net GPSRX: no longer DUE1.TX1
- net GPSTX: no longer DUE1.RX1
- net LED1: no longer DUE1.12
- net LED2: no longer DUE1.11
- net LEDB: no longer DUE1.A8, J3.P$4, X1-1.S
- net MAX1932!CL: no longer DUE1.3
- net MAX1932!CS1: no longer DUE1.TX3
- net MAX1932!CS2: no longer DUE1.RX3
- net MAX1932DIN: no longer DUE1.TX2
- net MAX1932SCLK: no longer DUE1.RX2
- net N$1: no longer X2-4.S
- net N$2: now also C69.2, U$10.PH0_XI, X2.P$1; no longer L1.1, X2-3.S
- net N$8: now also C70.2, U$10.PH1_XO, X2.P$2; no longer R4.1, R5.1, X3-1.S
- net PSUF1: now also C65.2, C66.2, C67.2, C68.2, U3.AO, U3.VDD, U4.VDD
- net RX0: no longer DUE1.RX0
- net SCL0: now also U3.SCL, U4.SCL; no longer DUE1.SCL
- net SDA0: now also U3.SDA, U4.SDA; no longer DUE1.SDA
- net SIG2A: no longer X1-2.S
- net SIG2B: now also IC$3.INB+; no longer X1-4.S
- net STRIGAOUT: no longer DUE1.A5
- net STRIGBOUT: no longer DUE1.A0
- net TRIGOUT: no longer DUE1.5
- net TX0: no longer DUE1.TX0
- net UCDAC0: now also U3.VOUT; no longer DUE1.DAC0
- net UCDAC1: now also U4.VOUT; no longer DUE1.DAC1
- net VBIAS1: no longer J4.P$3, X2-2.S
- net VBIAS2: no longer J4.P$4, X2-1.S
- net VBIASFB1: no longer DUE1.A3
- net VBIASFB2: no longer DUE1.A4
Other:
- note added: "Connections to Page 2"
- note removed: "Analogue Front End Interface 2 Molex KK 254 female sockets or RS Pro 2.54mm connectors"
- note removed: "DAC0 and DAC1 from the DUE are used to generate the reference levels. Voltages: 0.55V to 2.75V with 12 bit resolution."
- note removed: "GND_s"
- note removed: "Molex KK 254 series connectors."
- moved on the sheet: C2, C21, C22, C26, C27, C28, C29, C3, C30, C31, C32, C33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

Commit message: Updated schematic - nearly finished
Parts:
- removed J10, J11: 2p-2.54, Seeed-Connector:DIP-BLACK-MALE-HEADER-VERT(2P-2.54)
- removed R44, R45, R46: 1M, resistor:R-EU_R0603
- removed R48: 24.9k, resistor:R-EU_R0603
- removed R51: 15k, resistor:R-EU_R0603
- removed SIPM1, SIPM1_TOP, SIPM2, SIPM2_TOP: (no value), diode:DIODE-ADVANSID
- removed U5, U6: MAX1932, TQFN-12:MAX1932
- removed X4: 22-23-2051, con-molex:22-23-2051
- added C72, C75: 1n, rcl:C-EUC0603
- added C73, C74, C76: 100n, resistor:C-EUC0603
- added C77, C78: 20p, rcl:C-EUC0603
- added C79: 4.7u, resistor:C-EUC0603
- added D6: CD1206-S01575, diode:DIODE-MINIMELF
- added D7, D8: SS1P3L, SmartPrj:SS1P3L
- added IC10: AD8039, Cosmic Pi V2:ANALOG-DEVICES_AD8033R
- added IC11: 24C00OT, microchip:24C00OT
- added IC12: NCP1117ST33T3G -3V3, linear:MC33269ST-3.3T3
- added IC13: LM2734Y, SmartPrj:LM2736Y
- added J12, J13, J15, J16: 2p-2.54, Seeed-Connector:DIP-BLACK-MALE-HEADER-VERT(2P-2.54)
- added J14, J6: 2X4P-2.54, Seeed-Connector:DIP-BLACK-FEMALE-HEADER(2X4P-2.54)
- added J3, J4: BNCPTH, SparkFun-Connectors:BNCPTH
- added L10: MH2029-300Y, wuerth-elektronik:WE-CBF_0805
- added L11: 10u SRR0604-100ML, SmartPrj:L-USSRR0604
- added PC1, PC2: 47u, rcl:CPOL-EUD
- added PI_GPIO: (no value), con-lstb:MA20-2
- added R64, R73: 100, rcl:R-EU_R0603
- added R65, R74: 500k, rcl:R-EU_R0603
- added R66, R75: 1M, rcl:R-EU_R0603
- added R67, R68: 10K, rcl:R-EU_R0805
- added R69, R72: 0 ohm, rcl:R-EU_R1206
- added R70, R76: DNP, rcl:R-EU_R0603
- added R71, R77: 50k, rcl:R-EU_R0603
- added SIPM1X1_BOT, SIPM1X1_TOP: (no value), Cosmic Pi V2:DIODE_DIODE-ADVANSID1X1
- added SIPM3X3_BOT, SIPM3X3_TOP: (no value), Cosmic Pi V2:DIODE_DIODE-ADVANSID3X3
- added U$11: 310010495_STM32F401RET6, Seeed-OPL-2017-01-IC-Akita:310010495_STM32F401RET6
- added U$9: UCC27528UCC27528DR, Cosmic Pi V2:UCC27528UCC27528DR
- added X1: POWERSUPPLY_DC21MMX, SmartPrj:POWERSUPPLY_DC21MMX
- added X3: 306010282_XTAL_8MHZ-HC49US, Seeed-OPL-2017-01-Crystal-Akita:306010282_XTAL_8MHZ-HC49US
- C10: value 220n -> 100n; device rcl:C-EUC0603 -> resistor:C-EUC0603
- C45: value 220n -> 10u; device rcl:C-EUC0603 -> rcl:CPOL-EUSMCB
- C47: value 1u -> 10u; device resistor:C-EUC0603 -> rcl:CPOL-EUSMCB
- C48: value 100n -> 10n; device resistor:C-EUC0603 -> SmartPrj:C-EUC0603
- R10: value 1M -> 806
- R12: value 15k -> 806
- R13: value 1M -> 10k; device resistor:R-EU_R0603 -> SmartPrj:R-EU_R0402
- R14: value 1M -> 10K; device resistor:R-EU_R0603 -> SmartPrj:R-EU_0603-RND
- R19: value 24.9k -> 52K3; device resistor:R-EU_R0603 -> SmartPrj:R-EU_0603-RND
Connections:
- removed net !RESET: X4-4.S
- removed net MAX1932!CL: U5.!CL, U6.!CL
- removed net MAX1932!CS1: R10.2, U5.!CS
- removed net MAX1932!CS2: R44.2, U6.!CS
- removed net MAX1932DIN: R14.2, R46.2, U5.DIN, U6.DIN
- removed net MAX1932SCLK: R13.2, R45.2, U5.SCLK, U6.SCLK
- removed net N$17: BAT46WH1.K, C9.1, R20.2, U5.CS+
- removed net N$35: R51.1, U6.COMP
- removed net N$36: C45.1, R51.2
- removed net N$37: R48.2, R49.1, R50.2, U6.FB
- removed net N$54: R19.1, U5.DACOUT
- removed net N$56: C10.1, R12.2
- removed net RX0: X4-3.S
- removed net TX0: X4-2.S
- new net +4.1V: R67.1
- new net BOOST: C48.1, D6.C, IC13.BOOST
- new net BOOT1: PI_GPIO.7, U$10.BOOT0
- new net BOOT2: PI_GPIO.11, U$11.BOOT0
- new net EN: IC13.EN, R13.2
- new net FB: IC13.FB, R14.1, R19.2
- new net HV1EN: U$9.ENA
- new net HV1PWM: U$10.PA8, U$9.INA
- new net HV2EN: U$9.ENB
- new net HV2PWM: U$10.PA9, U$9.INB
- new net ID_SC: IC11.SCL, PI_GPIO.28
- new net ID_SD: IC11.SDA, PI_GPIO.27
- new net N$12: C72.1, IC10A.IN+, R64.2, R65.1
- new net N$52: C73.1, IC10A.IN-, R69.2
- new net N$59: C75.1, IC10B.IN+, R73.2, R74.1
- new net N$75: BAT46WH1.K, C9.1, R20.2
- new net N$76: J3.GND, R71.1
- new net N$77: C75.2, IC10B.OUT, R74.2, R75.1
- new net N$79: C77.2, U$11.PH0_XI, X3.P$1
- new net N$80: C74.1, IC10B.IN-, R72.2
- new net N$81: C78.2, U$11.PH1_XO, X3.P$2
- new net N$82: U$11.VSSA
- new net N$83: U$11.VSS1
- new net N$84: U$11.VSS2
- new net N$85: C79.2, U$11.VCAP
- new net NRST1: J12.1, U$10.NRST
- new net NRST2: U$11.NRST
- new net PSUFB1: R11.2, R21.1, U$10.PA0
- new net PSUFB2: R49.1, R50.2, U$10.PA1
- new net RESET: PI_GPIO.18
- new net SCL1: PI_GPIO.5
- new net SLOWAOUT: J3.OUT, R66.2, U$11.PA0
- new net SLOWBOUT: J4.OUT, R75.2, U$11.PA1
- new net SLOWCHA: C16.2, R26.1, R64.1
- new net SLOWCHB: C1.2, R17.1, R73.1
- new net SPI1_CLK: J13.2, U$11.PA5
- new net SPI1_MISO: U$10.PA6, U$11.PA6
- new net SPI1_MOSI: U$10.PA7, U$11.PA7
- new net SPI_CE0: PI_GPIO.24
- new net SPI_CE1: PI_GPIO.26
- new net STAGE3_DC_OFFSET: R67.2, R68.2, R69.1, R72.1
- new net SW: C48.2, D7.K, IC13.SW, L11.1
- new net TCK: PI_GPIO.23
- new net TCK/SWCLK1: J6.4, U$10.PA14
- new net TCK/SWCLK2: J14.4, U$11.PA14
- new net TDI: PI_GPIO.19
- new net TDI1: J6.6, U$10.PA15
- new net TDI2: J14.6, U$11.PA15
- new net TDO: PI_GPIO.21
- new net TDO/SWO1: J13.1, J6.5, U$10.PB3
- new net TDO/SWO2: J14.5, U$11.PB3
- new net TMS: PI_GPIO.22
- new net TMS/SWIDO1: J6.3, U$10.PA13
- new net TMS/SWIDO2: J14.3, U$11.PA13
- new net TRST1: J12.2, J6.7, U$10.PB4
- new net TRST2: J14.7, U$11.PB4
- new net VIN: C47.+, D8.K, IC13.VIN, PC1.+, R13.1
- new net VIN+: L10.2, X1.2
- net +3V3: now also C10.2, C45.+, IC11.VCC, IC12.OUT, IC12.OUT@1, J14.1, J6.1, U$10.VBAT, U$10.VDD1, U$10.VDD2, U$11.VBAT, U$11.VDD, U$11.VDD1, U$11.VDD2, U$11.VDD3, U$11.VDDA
- net +4V: now also C76.1, IC10P.V+
- net +5V: now also D6.A, IC12.IN, L11.2, PC2.+, PI_GPIO.2, PI_GPIO.4, R19.1, U$9.VDD; no longer C47.1, C48.1, R10.1, R44.1, U5.VIN, U6.VIN, X4-1.S
- net ACCELINT1: now also U$11.PC1
- net ACCELINT2: now also U$11.PC2
- net ACCELINT3: now also U$11.PC3
- net ACCELSA0: now also U$11.PC4
- net ACCELSA1: now also U$11.PC5
- net AGND: now also C73.2, C74.2, C76.2, IC10P.V-, R68.1, R70.1, R71.2, R76.1, R77.2
- net GND: now also C10.1, C45.-, C47.-, C70.1, C77.1, C78.1, C79.1, D7.A, IC11.GND, IC12.GND/ADJ, IC13.GND, J14.2, J14.8, J6.2, J6.8, PC1.-, PC2.-, PI_GPIO.14, PI_GPIO.20, PI_GPIO.25, PI_GPIO.30, PI_GPIO.34, PI_GPIO.39, PI_GPIO.6, PI_GPIO.9, R14.2, U$11.VSS, U$11.VSS3, U$9.GND, X1.1, X1.3; no longer C10.2, C45.2, C47.2, C48.2, J10.2, J11.2, R13.1, R14.1, R45.1, R46.1, U5.GND, U6.GND, X4-5.S
- net GPSRX: now also PI_GPIO.8
- net GPSTX: now also PI_GPIO.10
- net LEDB: now also U$10.PA5; no longer J10.1, J11.1
- net N$18: now also SIPM1X1_TOP.C, SIPM3X3_TOP.C; no longer SIPM1.C, SIPM1_TOP.C
- net N$19: now also R10.1; no longer U5.GATE
- net N$24: now also J4.GND, R77.1; no longer C1.2, R17.1
- net N$27: now also R12.1; no longer U6.GATE
- net N$30: no longer U6.CS+
- net N$32: now also C72.2, IC10A.OUT, R65.2, R66.1; no longer C16.2, R26.1
- net N$34: now also R12.2, U$9.OUTB; no longer R48.1, U6.DACOUT
- net N$47: now also R10.2, U$9.OUTA; no longer R11.2, R19.2, R21.1, U5.FB
- net N$55: now also D8.A, L10.1; no longer R12.1, U5.COMP
- net N$7: now also SIPM1X1_BOT.C, SIPM3X3_BOT.C; no longer SIPM2.C, SIPM2_TOP.C
- net SDA0: now also PI_GPIO.3
- net SIG1A: now also SIPM1X1_TOP.A, SIPM3X3_TOP.A; no longer SIPM1.A, SIPM1_TOP.A
- net SIG1B: now also SIPM1X1_BOT.A, SIPM3X3_BOT.A; no longer SIPM2.A, SIPM2_TOP.A
- net STRIGAOUT: now also U$11.PA10
- net STRIGBOUT: now also U$11.PA11
- net TRIGOUT: now also U$11.PA8
- net VBIAS1: no longer U5.CS-
- net VBIAS2: no longer U6.CS-
Other:
- note added: "Changes in this release: Version 2 with STM32 replacing Arduino DUE."
- note added: "Filtered Power Supplies"
- note added: "General notes: Not quite finished yet! The Pi Header pins still need checking. The SPI communication from Pi-STM32 1-STM32 2 needs checking. The JTAG/SWI programming from the Pi needs checking; how to programme each STM32 individually? Basically everything needs a good check."
- note added: "I, II and III stage amplifier offset voltages"
- note added: "IF LM2736Y"
- note added: "JTAG/STLink"
- note added: "Modifications since version 2.X: Slow channel amplifiers added for ADC sampling; 1mm2 Advansid SiPM footprint added. Combined with Main Board onto single PCB."
- note added: "PSU Controller uC"
- note added: "Pi Connector & E2"
- note added: "Power Supply (copied from the Arduino DUE)"
- note added: "R25, R32, R33, R67, R68 - 0.1% 25 ppm/K thin film"
- note added: "R2=1K"
- note added: "R3=330R"
- note added: "Reset Bridge"
- note added: "SPI_CLK"
- note added: "Slave SPI device; program directly or via SPI from main uC/Pi via address"
- note added: "Slow Output"
- note added: "Trigger Block 1K and 100p for RC Constant on 555 timer."
- note removed: "ADAFRUIT Ultimate GPS Header v3"
- note removed: "Arduino DUE header"
- note removed: "Boost PSU control IC"
- note removed: "Changes in this release: I2C variable resistor removed, DAC is now used for threshold setting. Pi Header added for in-box Pi connection."
- note removed: "Component notes: The circuit is designed to be mounted on an Arduino/Genduino DUE device. All capacitors shall be 50V rated. All SMT passives will generally be 603 unless otherwise indicated. This schematic has been modified with the lessons learned so far. More lessons are not excluded from future revisions. MAX1932 feedback resistors are set for Hamamatsu SiPM voltages"
- note removed: "I and II stage amplifier offset voltages"
- note removed: "LED header"
- note removed: "Modifications since version 2.4: U.FL connector changed for new part."
- note removed: "Pi Interconnect header"
- note removed: "Power supply filter for Trigger"
- note removed: "R25, R32, R33 - 0.1% 25 ppm/K thin film"
- note removed: "Trigger JP6 and JP7 allow threshold injection. 1K and 100p for RC Constant on 555 timer."
- moved on the sheet: BAT46WH2, C10, C11, C13, C14, C15, C26, C27, C28, C29, C32, C34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

Commit message: PSU complete in schematic. CPU to do.
Parts:
- removed J12, J13, J15, J16: 2p-2.54, Seeed-Connector:DIP-BLACK-MALE-HEADER-VERT(2P-2.54)
- added C80, C81, C82, C84, C85, C86: 100n, resistor:C-EUC0603
- added C83: 1u, resistor:C-EUC0603
- added C87: 4.7u, resistor:C-EUC0603
- added D10, D9: GREEN-0603, Seeed-LED:SMD-LED-CLEAR-GREEN(0603)
- added JP1: JUMPER-SMT_3_1-NC_PASTE_SILK, SparkFun-Jumpers:JUMPER-SMT_3_1-NC_PASTE_SILK
- added R44, R45: 470, SmartPrj:R-EU_R0402
Connections:
- net RESET renamed CPU_BOOT1
- net TCK/SWCLK1 renamed PSU_JTCK-SWCLK
- net TDI1 renamed PSU_SYS_JTDI
- net TMS/SWIDO1 renamed PSU_JTMS-SWDIO
- removed net BOOT1: PI_GPIO.7, U$10.BOOT0
- removed net BOOT2: PI_GPIO.11, U$11.BOOT0
- removed net NRST1: J12.1, U$10.NRST
- removed net NRST2: U$11.NRST
- removed net SPI1_CLK: J13.2, U$11.PA5
- removed net SPI1_MISO: U$10.PA6, U$11.PA6
- removed net SPI1_MOSI: U$10.PA7, U$11.PA7
- removed net TCK: PI_GPIO.23
- removed net TCK/SWCLK2: J14.4, U$11.PA14
- removed net TDI: PI_GPIO.19
- removed net TDI2: J14.6, U$11.PA15
- removed net TDO: PI_GPIO.21
- removed net TDO/SWO1: J13.1, J6.5, U$10.PB3
- removed net TDO/SWO2: J14.5, U$11.PB3
- removed net TMS: PI_GPIO.22
- removed net TMS/SWIDO2: J14.3, U$11.PA13
- removed net TRST1: J12.2, J6.7, U$10.PB4
- removed net TRST2: J14.7, U$11.PB4
- new net CPU_NRST: PI_GPIO.16
- new net N$35: D9.+, R44.2
- new net N$36: R44.1, U$10.PC0
- new net N$54: R45.1, U$11.PC0
- new net N$61: D10.+, R45.2
- new net PSU_BOOT0: PI_GPIO.13
- new net PSU_JTDO-SWO: J6.8, U$10.PB3
- new net PSU_NRST: C80.1, J6.5, PI_GPIO.11, U$10.NRST
- new net PSU_SYS_JTRST: J6.7, U$10.PB4
- new net SPI_CLK: PI_GPIO.23, U$10.PA5
- new net SPI_MISO: PI_GPIO.21, U$10.PA6
- new net SPI_MOSI: PI_GPIO.19, U$10.PA7
- new net TM1LEDB: JP1.1, U$10.PA10
- new net TM3LEDB: JP1.3, U$10.PC6
- net +3V3: now also C81.1, C82.1, C83.1, C84.1, C85.1, C86.1, C87.1; no longer J14.1
- net ACCELINT1: no longer U$11.PC1
- net ACCELINT2: no longer U$11.PC2
- net ACCELINT3: no longer U$11.PC3
- net ACCELSA0: no longer U$11.PC4
- net ACCELSA1: no longer U$11.PC5
- net GND: now also C80.2, C81.2, C82.2, C83.2, C84.2, C85.2, C86.2, C87.2, D10.-, D9.-; no longer J14.8, J6.8
- net HV1EN: now also U$10.PB0
- net HV1PWM: now also U$10.PA0; no longer U$10.PA8
- net HV2EN: now also U$10.PB1
- net HV2PWM: now also U$10.PA3; no longer U$10.PA9
- net LEDB: now also JP1.2; no longer U$10.PA5
- net PSUFB1: now also U$10.PA1; no longer U$10.PA0
- net PSUFB2: now also U$10.PA2; no longer U$10.PA1
- net SLOWAOUT: no longer U$11.PA0
- net SLOWBOUT: no longer U$11.PA1
- net SPI_CE1: now also U$10.PA4
- net STRIGAOUT: no longer U$11.PA10
- net STRIGBOUT: no longer U$11.PA11
- net TRIGOUT: no longer U$11.PA8
Other:
- note removed: "Reset Bridge"
- note removed: "SPI_CLK"
- moved on the sheet: J6

Commit message: Schematic design completed.
PSU + CPU outputs changed a little after reading the STM32 manual
Parts:
- removed JP1: JUMPER-SMT_3_1-NC_PASTE_SILK, SparkFun-Jumpers:JUMPER-SMT_3_1-NC_PASTE_SILK
- added C88, C90, C91, C92, C93, C94: 100n, resistor:C-EUC0603
- added C89: 4.7u, resistor:C-EUC0603
- added C95: 1u, resistor:C-EUC0603
- added CN1: 6p-2.54, Seeed-Connector:DIP-BLACK-FEMALE-HEADER-VERT(6P-2.54)
- R44, R45: value 470 -> 40; device SmartPrj:R-EU_R0402 -> resistor:R-EU_R0603
Connections:
- removed net +4.1V: R67.1
- removed net AMP2A: IC$3.INA+
- removed net CPU_BOOT1: PI_GPIO.18
- removed net N$61: D10.+, R45.2
- removed net N$82: U$11.VSSA
- removed net N$83: U$11.VSS1
- removed net N$84: U$11.VSS2
- removed net SCL1: PI_GPIO.5
- removed net TM1LEDB: JP1.1, U$10.PA10
- removed net TM3LEDB: JP1.3, U$10.PC6
- new net CPU_BOOT0: PI_GPIO.18, U$11.BOOT0
- new net CPU_JTCK-SWCLK: J14.4, U$11.PA14
- new net CPU_JTDO-SWO: J14.8, U$11.PB3
- new net CPU_JTMS-SWDIO: J14.3, U$11.PA13
- new net CPU_SYS_JTDI: J14.6, U$11.PA15
- new net CPU_SYS_JTRST: J14.7, U$11.PB4
- new net N$71: C91.1, C95.1, U$11.VDDA
- new net N$78: C89.1, C90.1, U$11.VBAT, U$11.VDD
- new net PI_FLAG0: PI_GPIO.7, U$11.PC8
- new net PI_FLAG1: PI_GPIO.12, U$11.PC9
- new net PI_FLAG2: PI_GPIO.15, U$11.PC10
- new net USER_0: CN1.3, U$11.PC11
- new net USER_1: CN1.4, U$11.PC12
- new net USER_2: CN1.5, U$11.PC13
- new net USER_3: CN1.6, U$11.PC14
- net +3V3: now also CN1.1, J14.1; no longer U$11.VBAT, U$11.VDD, U$11.VDD1, U$11.VDD2, U$11.VDD3, U$11.VDDA
- net +4V: now also R67.1
- net +5V: now also L1.4
- net ACCELINT1: now also U$11.PC3
- net ACCELINT2: now also U$11.PC4
- net ACCELINT3: now also U$11.PC5
- net ACCELSA0: now also U$11.PC6
- net ACCELSA1: now also U$11.PC7
- net CPU_NRST: now also C88.1, J14.5, U$11.NRST
- net GND: now also C88.2, C89.2, C90.2, C91.2, C92.2, C93.2, C94.2, C95.2, CN1.2, U$10.VSS1, U$10.VSS2, U$10.VSSA, U$11.VSS1, U$11.VSS2, U$11.VSSA
- net GPSPPS: now also U$11.PA8
- net HV1EN: now also U$10.PC1; no longer U$10.PB0
- net HV2EN: now also U$10.PC2; no longer U$10.PB1
- net LED1: now also U$11.PC1
- net LED2: now also U$11.PC2
- net LEDB: now also U$10.PA8; no longer JP1.2
- net N$1: now also D10.+, R44.2; no longer L1.4
- net N$21: now also C94.1, U$11.VDD3; no longer U$10.VSSA
- net N$35: now also R45.2; no longer R44.2
- net N$36: now also R45.1; no longer R44.1
- net N$49: now also C93.1, U$11.VDD2; no longer U$10.VSS1
- net N$51: now also C92.1, U$11.VDD1; no longer U$10.VSS2
- net N$54: now also R44.1; no longer R45.1
- net SCL0: now also PI_GPIO.5
- net SIG2A: now also IC$3.INA+
- net SLOWAOUT: now also R70.2, U$11.PA1
- net SLOWBOUT: now also R76.2, U$11.PA2
- net SPI_CE0: now also U$11.PA4
- net SPI_CLK: now also U$11.PA5
- net SPI_MISO: now also U$11.PA6
- net SPI_MOSI: now also U$11.PA7
- net STRIGAOUT: now also U$11.PA10
- net STRIGBOUT: now also U$11.PA11
- net TRIGOUT: now also U$11.PA9
Other:
- note removed: "+V_s"
- moved on the sheet: D10, D9, J14, R44, R45, R70, R76

Commit message: schematic complete, layout tweaks and routing required
Parts:
- removed C48: 10n, SmartPrj:C-EUC0603
- removed PI_GPIO: (no value), con-lstb:MA20-2
- added LED3: top-mounted, eagle-ltspice:LED_ESML0603
- added LED4: bottom-mounted, eagle-ltspice:LED_ESML0603
- added R46: top-mounted, rcl:R-US_R0402
- added R48: bottom-mounted, rcl:R-US_R0402
- added U$12: RPI-ZERO, RPI-Zero:RPI-ZERO
- added USB1: 10118193-0001LF, Seeed-Connector:MICRO-USB-SMD-B-(10118193-0001LF)
- J3, J4: value BNCPTH -> 5-1814400-1_5-1814400-1; device SparkFun-Connectors:BNCPTH -> Cosmic Pi V2:5-1814400-1_5-1814400-1
- R13: value 10k -> 10K; device SmartPrj:R-EU_R0402 -> Seeed-Resistor:SMD-RES-10K-1%-1/10W(0603)
- R14: device SmartPrj:R-EU_0603-RND -> Seeed-Resistor:SMD-RES-10K-1%-1/10W(0603)
- R19: value 52K3 -> 51K; device SmartPrj:R-EU_0603-RND -> Seeed-Resistor:SMD-RES-51K-5%-1/10W(0603)
- renumbered U$10 to PSU, U$11 to CPU
Connections:
- new net 5V0@2: U$12.5V0@1, U$12.5V0@2
- new net GND@3: U$12.GND@1, U$12.GND@2, U$12.GND@3
- new net GND@7: U$12.GND@4, U$12.GND@5, U$12.GND@6, U$12.GND@7, U$12.GND@8
- net +5V: now also USB1.VCC; no longer PI_GPIO.2, PI_GPIO.4
- net AGND: now also LED3.C, LED4.C
- net BOOST: no longer C48.1
- net CPU_BOOT0: now also U$12.GEN5/GPIO24; no longer PI_GPIO.18
- net CPU_NRST: now also U$12.GEN4/GPIO23; no longer PI_GPIO.16
- net GND: now also USB1.GND@1, USB1.GND@2, USB1.GND@3, USB1.GND@4, USB1.GND@5; no longer PI_GPIO.14, PI_GPIO.20, PI_GPIO.25, PI_GPIO.30, PI_GPIO.34, PI_GPIO.39, PI_GPIO.6, PI_GPIO.9
- net GPSRX: now also U$12.TXD0/GPIO14; no longer PI_GPIO.8
- net GPSTX: now also U$12.RXD0/GPIO15; no longer PI_GPIO.10
- net ID_SC: now also U$12.ID_SC; no longer PI_GPIO.28
- net ID_SD: now also U$12.ID_SD; no longer PI_GPIO.27
- net N$20: now also LED3.A
- net N$24: now also J4.GND@1; no longer J4.GND
- net N$3: now also LED4.A
- net N$76: now also J3.GND@1; no longer J3.GND
- net PI_FLAG0: now also U$12.GPIO4/GCKL; no longer PI_GPIO.7
- net PI_FLAG1: now also U$12.GPIO18; no longer PI_GPIO.12
- net PI_FLAG2: now also U$12.GPIO22/GEN3; no longer PI_GPIO.15
- net PSU_BOOT0: now also U$12.GPIO27/GEN2; no longer PI_GPIO.13
- net PSU_NRST: now also U$12.GPIO17/GEN0; no longer PI_GPIO.11
- net SCL0: now also U$12.GPIO3/SCL1; no longer PI_GPIO.5
- net SDA0: now also U$12.GPIO2/SDA1; no longer PI_GPIO.3
- net SLOWAOUT: now also J3.SIG; no longer J3.OUT
- net SLOWBOUT: now also J4.SIG; no longer J4.OUT
- net SPI_CE0: now also U$12.!CE0!/GPIO8; no longer PI_GPIO.24
- net SPI_CE1: now also U$12.!CE!/GPIO7; no longer PI_GPIO.26
- net SPI_CLK: now also U$12.GPIO11/SCLK; no longer PI_GPIO.23
- net SPI_MISO: now also U$12.GPIO9/MISO; no longer PI_GPIO.21
- net SPI_MOSI: now also U$12.GPIO10/MOSI; no longer PI_GPIO.19
- net SW: no longer C48.2
- net TEMP1: now also R46.1, R48.1
- net TEMP2: now also R46.2, R48.2
Other:
- note added: "Changes in this release: Version 2 with STM32 replacing Arduino DUE. Designed to fit as a PiHat for a Pi Zero W."
- note added: "Modules: Page 1 - Amplifiers A&B Slow output amplifiers A&B Page 2 - HV PSU (A&B) GPS (L70 or L76) Accelerometer & Altimeter Humidity & Temperature Power Filter Discriminator Trigger Indicator LEDs STM32 modules"
- note added: "N. Beev, J. Devine Team Cosmic Pi 29/04/18 Version 2.5 Released under CERN OHL V1.2"
- note added: "Released under CERN OHL V1.2 29/04/18"
- note removed: "Changes in this release: Version 2 with STM32 replacing Arduino DUE."
- note removed: "General notes: Not quite finished yet! The Pi Header pins still need checking. The SPI communication from Pi-STM32 1-STM32 2 needs checking. The JTAG/SWI programming from the Pi needs checking; how to programme each STM32 individually? Basically everything needs a good check."
- note removed: "J. Devine, C. Cantini, N. Beev Team Cosmic Pi 06.10.2017 Version 2.5 Released under CERN OHL V1.2"
- note removed: "Modules: Input (A&B) HV PSU (A&B) GPS (L70 or L76) Accelerometer & Altimeter Humidity & Temperature Power Filter Discriminator Trigger Indicator LEDs"
- note removed: "Released under CERN OHL V1.2 05/10/17"
- moved on the sheet: LED1, LED2, R19, R5, R70, R71, R76, R77
