File: Cosmic Pi V2.sch (EAGLE design)
At the start: 252 parts, among them CN1 6p-2.54, IC1 AD8039, IC10 AD8039, IC11 24C00OT, IC12 NCP1117ST33T3G -3V3, IC13 LM2734Y, IC2 AD8039, IC3 LP2985IM5-3.1, IC4 LM555D, IC5 LM555D, IC6 LM555D, IC7 74AUC1G00DBV, IC8 74AUC1G00DBV, IC9 74AUC1G00DBV, J1 U.FL-R-SMT-1(10), J14 2X4P-2.54, J2 U.FL-R-SMT-1(10), J3 5-1814400-1_5-1814400-1, J4 5-1814400-1_5-1814400-1, J5 5-1814400-1, J6 2X4P-2.54, J7 2p-2.54, J8 2p-2.54, J9 2p-2.54, Q1 BSS123, Q2 BSS123, U1 L76-M33, U2 LSM303D, U3 MCP4725, U4 MCP4725, X1 POWERSUPPLY_DC21MMX, X2 306010282_XTAL_8MHZ-HC49US, X3 306010282_XTAL_8MHZ-HC49US

Commit message: Update following testing of 4 prototypes.
 Note .BRD isn't updated.
Parts:
- removed BAT46WH1, BAT46WH2: BAT46WH, BAT46Wsymbol:BAT46WH
- removed C69, C70: 20p, rcl:C-EUC0603
- removed CN1: 6p-2.54, Seeed-Connector:DIP-BLACK-FEMALE-HEADER-VERT(6P-2.54)
- removed IC$1: LPS25H, LPS25H:LPS25H
- removed IC$2: SI7006A20, SI7006:SI7006A20
- removed J14: 2X4P-2.54, Seeed-Connector:DIP-BLACK-FEMALE-HEADER(2X4P-2.54)
- removed J7, J8, J9: 2p-2.54, Seeed-Connector:DIP-BLACK-MALE-HEADER-VERT(2P-2.54)
- removed LED1, LED3: top-mounted, eagle-ltspice:LED_ESML0603
- removed LED2, LED4: bottom-mounted, eagle-ltspice:LED_ESML0603
- removed R33: 10K, rcl:R-EU_R0805
- removed R44: 40, resistor:R-EU_R0603
- removed R46: top-mounted, rcl:R-US_R0402
- removed R48: bottom-mounted, rcl:R-US_R0402
- removed R69, R72: 0 ohm, rcl:R-EU_R1206
- removed R70, R76: DNP, rcl:R-EU_R0603
- removed U$12: RPI-ZERO, RPI-Zero:RPI-ZERO
- removed U2: LSM303D, LSM303D:LSM303D
- removed X3: 306010282_XTAL_8MHZ-HC49US, Seeed-OPL-2017-01-Crystal-Akita:306010282_XTAL_8MHZ-HC49US
- added C48: 10n, resistor:C-EUC0603
- added D11: GREEN-0603, Seeed-LED:SMD-LED-CLEAR-GREEN(0603)
- added D12: BLUE-0402, Seeed-LED:SMD-LED-CLEAR-BLUE(0402)
- added D13, D14: BAT46WH, BAT46Wsymbol:BAT46WH
- added D15: SS1P3L, SmartPrj:SS1P3L
- added IC14: LPS25H, LPS25H:LPS25H
- added IC15: SI7006A20, SI7006:SI7006A20
- added IC16: LSM303D, LSM303D:LSM303D
- added X4, X5: 1296-T08, con-leotronics:1296-T08
- C45, C47: value 10u -> 10uf; device rcl:CPOL-EUSMCB -> Seeed-Capacitor:TANTALUM-SMD-10UF-16V-10%(AVX-A)
- D1: value L-710A8GE/1I1GD-RV -> BLUE-0603; device KingbriteBiLevel T1:KINGBRITET1 -> Seeed-LED:SMD-LED-CLEAR-BLUE(0603)
- D10: value GREEN-0603 -> BLUE-0402; device Seeed-LED:SMD-LED-CLEAR-GREEN(0603) -> Seeed-LED:SMD-LED-CLEAR-BLUE(0402); POSITION (none) -> TOP Mount
- IC1: value AD8039 -> AD8039R; device analog-devices:AD8033R -> cosmicanalogue:AD8039R; MF Analogue Devices -> (none); MPN AD8039ARZ -> (none); OC_FARNELL 2727242RL -> (none); OC_NEWARK na -> (none)
- IC10: value AD8039 -> AD8039R; device Cosmic Pi V2:ANALOG-DEVICES_AD8033R -> cosmicanalogue:AD8039R
- IC2: value AD8039 -> AD8039R; device analog-devices:AD8033R -> cosmicanalogue:AD8039R; MF Analouge Devices -> (none); MPN AD8039ARZ -> (none); OC_FARNELL 2727242RL -> (none); OC_NEWARK na -> (none)
- J6: value 2X4P-2.54 -> CONN_20X2SHROUDED_SMT; device Seeed-Connector:DIP-BLACK-FEMALE-HEADER(2X4P-2.54) -> SparkFun-Connectors:CONN_20X2SHROUDED_SMT
- R1: value 1k -> 1K
- R10, R12, R20, R47: value 806 -> 820
- R17, R26: value 1K -> 1k
- R19: value 51K -> 51k
- R25: value 10K -> 100K; device rcl:R-EU_R0805 -> rcl:R-EU_R0603
- R34, R35, R45: value 40 -> 330
- R4: value top-mounted -> 10K; device rcl:R-US_R0402 -> rcl:R-EU_R0805
- R40: value 100k -> 100K
- R5: value bottom-mounted -> 100K; device rcl:R-US_R0402 -> rcl:R-EU_R0603
- R62, R63: value 330R -> 10k
- R66, R75: value 1M -> 10
- R71, R77: value 50k -> 1k
- R9: value 0 ohm -> 0
- X2: value 306010282_XTAL_8MHZ-HC49US -> 306010032_XTAL_8MHZ_5032_4P; device Seeed-OPL-2017-01-Crystal-Akita:306010282_XTAL_8MHZ-HC49US -> Seeed-OPL-2017-01-Crystal-Akita:306010032_XTAL_8MHZ_5032_4P
- renumbered U$9 to IC17
Connections:
- removed net 5V0@2: U$12.5V0@1, U$12.5V0@2
- removed net ACCELSA0: CPU.PC6, U2.SDO
- removed net ACCELSA1: CPU.PC7, IC$1.SA0
- removed net GND@3: U$12.GND@1, U$12.GND@2, U$12.GND@3
- removed net GND@7: U$12.GND@4, U$12.GND@5, U$12.GND@6, U$12.GND@7, U$12.GND@8
- removed net N$49: C93.1, CPU.VDD2
- removed net N$51: C92.1, CPU.VDD1
- removed net N$52: C73.1, IC10A.IN-, R69.2
- removed net N$54: CPU.PC0, R44.1
- removed net N$71: C91.1, C95.1, CPU.VDDA
- removed net N$78: C89.1, C90.1, CPU.VBAT, CPU.VDD
- removed net N$80: C74.1, IC10B.IN-, R72.2
- removed net STAGE1_DC_OFFSET: C19.1, C24.1, D3.A1, D3.C2, D4.A1, D4.C2, IC1A.IN+, IC2A.IN+, R25.2, R33.2
- removed net STAGE2_DC_OFFSET: C25.1, IC2B.IN+, R32.2, R33.1, R9.1
- removed net STAGE3_DC_OFFSET: R67.2, R68.2, R69.1, R72.1
- removed net TEMP1: R4.1, R46.1, R48.1, R5.1
- removed net TEMP2: R4.2, R46.2, R48.2, R5.2
- removed net USER_0: CN1.3, CPU.PC11
- removed net USER_1: CN1.4, CPU.PC12
- removed net USER_2: CN1.5, CPU.PC13
- removed net USER_3: CN1.6, CPU.PC14
- new net DC_OFFSET: C19.1, C24.1, C25.1, C73.1, C74.1, D3.A1, D3.C2, D4.A1, D4.C2, IC10A.IN+, IC10B.IN+, IC1A.IN+, IC2A.IN+, IC2B.IN+, R32.2, R68.2, R9.1
- new net N$10: D15.A, USB1.VCC
- net +3V3: now also C89.1, C90.1, C91.1, C92.1, C93.1, C94.1, C95.1, CPU.VBAT, CPU.VDD, CPU.VDD1, CPU.VDD2, CPU.VDD3, CPU.VDDA, IC14.CS, IC14.VDD, IC14.VDD_IO, IC15.VDD, IC16.CS, IC16.VDD, IC16.VDD_IO, X4-1.B, X5-1.B; no longer CN1.1, IC$1.CS, IC$1.VDD, IC$1.VDD_IO, IC$2.VDD, J14.1, J6.1, U2.CS, U2.VDD, U2.VDD_IO
- net +4V: now also R4.1; no longer R25.1, R67.1
- net +5V: now also D15.K, J6.2, J6.4; no longer USB1.VCC
- net ACCELINT1: now also IC16.INT1, J6.33; no longer CPU.PC3, U2.INT1
- net ACCELINT2: now also IC16.INT2, J6.35; no longer CPU.PC4, U2.INT2
- net ACCELINT3: now also IC14.INT, J6.37; no longer CPU.PC5, IC$1.INT
- net AGND: now also D10.-, D12.-; no longer LED1.C, LED2.C, LED3.C, LED4.C, R32.1, R70.1, R76.1
- net BOOST: now also C48.2
- net CPU_BOOT0: now also J6.18; no longer U$12.GEN5/GPIO24
- net CPU_JTCK-SWCLK: now also X4-7.B; no longer J14.4
- net CPU_JTDO-SWO: now also X4-2.B; no longer J14.8
- net CPU_JTMS-SWDIO: now also X4-5.B; no longer J14.3
- net CPU_NRST: now also J6.16, X4-8.B; no longer J14.5, U$12.GEN4/GPIO23
- net CPU_SYS_JTDI: now also X4-6.B; no longer J14.6
- net CPU_SYS_JTRST: now also X4-4.B; no longer J14.7
- net GND: now also D1.-, D11.-, IC14.GND@1, IC14.GND@2, IC14.RGND, IC14.SA0, IC15.GND, IC16.GND, IC16.RES, IC16.SDO, J6.14, J6.20, J6.25, J6.30, J6.34, J6.39, J6.6, J6.9, X2.GND1, X2.GND2, X4-3.B, X5-3.B; no longer C69.1, C70.1, CN1.2, D1.2, D1.4, D10.-, IC$1.GND@1, IC$1.GND@2, IC$1.RGND, IC$2.GND, J14.2, J6.2, J7.2, J8.2, J9.2, U2.GND, U2.RES
- net GPSPPS: now also CPU.PA0; no longer CPU.PA8
- net GPSRX: now also J6.8; no longer U$12.TXD0/GPIO14
- net GPSTX: now also J6.10; no longer U$12.RXD0/GPIO15
- net ID_SC: now also J6.28; no longer U$12.ID_SC
- net ID_SD: now also J6.27; no longer U$12.ID_SD
- net N$1: now also J3.SIG, R5.2; no longer D10.+, R44.2
- net N$12: now also IC10A.IN-; no longer IC10A.IN+
- net N$16: now also D13.A; no longer BAT46WH1.A
- net N$2: now also R4.2, R67.1; no longer C69.2, PSU.PH0_XI, X2.P$1
- net N$20: now also D10.+; no longer LED1.A, LED3.A
- net N$21: now also R32.1, R67.2; no longer C94.1, CPU.VDD3
- net N$28: now also D14.A; no longer BAT46WH2.A
- net N$3: now also D12.+; no longer LED2.A, LED4.A
- net N$30: now also D14.K; no longer BAT46WH2.K
- net N$59: now also IC10B.IN-; no longer IC10B.IN+
- net N$63: now also IC16.SETP; no longer U2.SETP
- net N$64: now also IC16.SETC; no longer U2.SETC
- net N$65: now also IC16.C1; no longer U2.C1
- net N$72: now also D1.+; no longer D1.1
- net N$73: now also D11.+; no longer D1.3
- net N$75: now also D13.K; no longer BAT46WH1.K
- net N$79: now also X2.P$2; no longer X3.P$1
- net N$8: now also J4.SIG, R25.2; no longer C70.2, PSU.PH1_XO, X2.P$2
- net N$81: now also X2.P$1; no longer X3.P$2
- net PI_FLAG0: now also J6.7; no longer U$12.GPIO4/GCKL
- net PI_FLAG1: now also J6.12; no longer U$12.GPIO18
- net PI_FLAG2: now also J6.15; no longer U$12.GPIO22/GEN3
- net PSU_BOOT0: now also J6.13, PSU.BOOT0; no longer U$12.GPIO27/GEN2
- net PSU_JTCK-SWCLK: now also X5-7.B; no longer J6.4
- net PSU_JTDO-SWO: now also X5-2.B; no longer J6.8
- net PSU_JTMS-SWDIO: now also X5-5.B; no longer J6.3
- net PSU_NRST: now also J6.11, X5-8.B; no longer J6.5, U$12.GPIO17/GEN0
- net PSU_SYS_JTDI: now also X5-6.B; no longer J6.6
- net PSU_SYS_JTRST: now also X5-4.B; no longer J6.7
- net SCL0: now also IC14.SCL, IC15.SCL, IC16.SCL/SPC, J6.5; no longer IC$1.SCL, IC$2.SCL, U$12.GPIO3/SCL1, U2.SCL/SPC
- net SDA0: now also IC14.SDA, IC15.SDA, IC16.SDA/SDI, J6.3; no longer IC$1.SDA, IC$2.SDA, U$12.GPIO2/SDA1, U2.SDA/SDI
- net SLOWAOUT: now also CPU.PA7, R5.1; no longer CPU.PA1, J3.SIG, R70.2
- net SLOWBOUT: now also CPU.PB0, R25.1; no longer CPU.PA2, J4.SIG, R76.2
- net SPI_CE0: now also J6.24; no longer U$12.!CE0!/GPIO8
- net SPI_CE1: now also J6.26; no longer U$12.!CE!/GPIO7
- net SPI_CLK: now also J6.23; no longer U$12.GPIO11/SCLK
- net SPI_MISO: now also J6.21; no longer U$12.GPIO9/MISO
- net SPI_MOSI: now also CPU.PB5, J6.19; no longer CPU.PA7, U$12.GPIO10/MOSI
- net STRIGAOUT: now also CPU.PB10; no longer CPU.PA10, J8.1
- net STRIGBOUT: now also CPU.PA3; no longer CPU.PA11, J9.1
- net SW: now also C48.1
- net TRIGOUT: now also CPU.PA1; no longer CPU.PA9, J7.1
Other:
- note added: "2 Page schematic by team Cosmic Pi."
- note added: "Changes in this release: Corrected pinout on CPU to use 32 bit timers. Corrected AD8039 pinout for slow channel amp. Added 10nF capacitor to level out 5V supply; measured at 4.88V on corrected hardware. Added reverse protection diode to 5V from USB."
- note added: "Main uC"
- note added: "Note Pi Zero Header is flipped, the Pi Zero is inserted upside down."
- note added: "R4, R67, R32, R68 - 0.1% 25 ppm/K thin film"
- note removed: "Changes in this release: Version 2 with STM32 replacing Arduino DUE. Designed to fit as a PiHat for a Pi Zero W."
- note removed: "Output headers"
- note removed: "R25, R32, R33, R67, R68 - 0.1% 25 ppm/K thin film"
- note removed: "Schematic by team Cosmic Pi"
- note removed: "Sensor: Murata NCP15XH103F03RC"
- note removed: "Temperature Sensor"
- moved on the sheet: C12, C13, C26, C27, C28, C29, C30, C31, C32, C33, C34, C35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
