File: Cosmic Pi V2.brd (EAGLE design)
At the start: 120 x 159.8 mm, 252 parts, among them CN1 6p-2.54, IC1 AD8039, IC10 AD8039, IC11 24C00OT, IC12 NCP1117ST33T3G -3V3, IC13 LM2734Y, IC2 AD8039, IC3 LP2985IM5-3.1, IC4 LM555D, IC5 LM555D, IC6 LM555D, IC7 74AUC1G00DBV, IC8 74AUC1G00DBV, IC9 74AUC1G00DBV, J1 U.FL-R-SMT-1(10), J14 2X4P-2.54, J2 U.FL-R-SMT-1(10), J3 5-1814400-1_5-1814400-1, J4 5-1814400-1_5-1814400-1, J5 5-1814400-1, J6 2X4P-2.54, J7 2p-2.54, J8 2p-2.54, J9 2p-2.54, Q1 BSS123, Q2 BSS123, U1 L76-M33, U2 LSM303D, U3 MCP4725, U4 MCP4725, X1 POWERSUPPLY_DC21MMX, X2 306010282_XTAL_8MHZ-HC49US, X3 306010282_XTAL_8MHZ-HC49US

Commit message: Update following testing of 4 prototypes.
 Note .BRD isn't updated.
Parts:
- removed BAT46WH1, BAT46WH2: BAT46WH, BAT46Wsymbol:SOD123F
- removed C69, C70: 20p, rcl:C0603
- removed CN1: 6p-2.54, Seeed-Connector:H6-2.54
- removed IC$1: LPS25H, LPS25H:LPS25H
- removed IC$2: SI7006A20, SI7006:3X3DFN
- removed J14: 2X4P-2.54, Seeed-Connector:H2X4-2.54
- removed J7, J8, J9: 2p-2.54, Seeed-Connector:H2-2.54
- removed LED1, LED3: top-mounted, eagle-ltspice:LED_SML0603
- removed LED2, LED4: bottom-mounted, eagle-ltspice:LED_SML0603
- removed R33: 10K, rcl:R0805
- removed R44: 40, resistor:R0603
- removed R46: top-mounted, rcl:R0402
- removed R48: bottom-mounted, rcl:R0402
- removed R69, R72: 0 ohm, rcl:R1206
- removed R70, R76: DNP, rcl:R0603
- removed U$12: RPI-ZERO, RPI-Zero:RASPBERRYPI_BASTELSTUBE_V13_RASPI_BOARD_B+_FULL
- removed U$9: UCC27528UCC27528DR, Cosmic Pi V2:ANALOG-DEVICES_SO8
- removed U2: LSM303D, LSM303D:LGA16L
- removed X3: 306010282_XTAL_8MHZ-HC49US, Seeed-OPL-2017-01-Crystal-Akita:HC49UP
- added C48: 10n, resistor:C0603
- added D11: GREEN-0603, Seeed-LED:LED-0603
- added D12: BLUE-0402, Seeed-LED:LED-0402
- added D13, D14: BAT46WH, BAT46Wsymbol:SOD123F
- added D15: SS1P3L, SmartPrj:DO220AAL
- added IC14: LPS25H, LPS25H:LPS25H
- added IC15: SI7006A20, SI7006:3X3DFN
- added IC16: LSM303D, LSM303D:LGA16L
- added IC17: UCC27528UCC27528DR, Cosmic Pi V2:ANALOG-DEVICES_SO8
- added X4, X5: 1296-T08, con-leotronics:1296-08
- C45, C47: value 10u -> 10uf; device rcl:SMC_B -> Seeed-Capacitor:AVX-A
- D1: value L-710A8GE/1I1GD-RV -> BLUE-0603; device KingbriteBiLevel T1:2X02 -> Seeed-LED:LED-0603
- D10: value GREEN-0603 -> BLUE-0402; device Seeed-LED:LED-0603 -> Seeed-LED:LED-0402
- IC1, IC2: value AD8039 -> AD8039R; device analog-devices:SO8 -> cosmicanalogue:SO8
- IC10: value AD8039 -> AD8039R; device Cosmic Pi V2:ANALOG-DEVICES_SO8 -> cosmicanalogue:SO8
- J6: value 2X4P-2.54 -> CONN_20X2SHROUDED_SMT; device Seeed-Connector:H2X4-2.54 -> SparkFun-Connectors:2X20_SHROUDED_SMT
- R1: value 1k -> 1K
- R10, R12, R20, R47: value 806 -> 820
- R17, R26: value 1K -> 1k
- R19: value 51K -> 51k
- R25: value 10K -> 100K; device rcl:R0805 -> rcl:R0603
- R34, R35, R45: value 40 -> 330
- R4: value top-mounted -> 10K; device rcl:R0402 -> rcl:R0805
- R40: value 100k -> 100K
- R5: value bottom-mounted -> 100K; device rcl:R0402 -> rcl:R0603
- R62, R63: value 330R -> 10k
- R66, R75: value 1M -> 10
- R71, R77: value 50k -> 1k
- R9: value 0 ohm -> 0
- X2: value 306010282_XTAL_8MHZ-HC49US -> 306010032_XTAL_8MHZ_5032_4P; device Seeed-OPL-2017-01-Crystal-Akita:HC49UP -> Seeed-OPL-2017-01-Crystal-Akita:X5032_4P
- moved IC10 112.5 mm to (4.42, -26.5), turned to 0 degrees
- moved IC2 109.1 mm to (4.42, -45.1), turned to 0 degrees
- moved IC1 84.6 mm to (4.42, -35.8), turned to 0 degrees
- moved C77 75.7 mm to (31.8, 4.50), flipped to the top
- moved L1 75.0 mm to (98.0, 18.2), flipped to the bottom
- moved L4 73.7 mm to (102.6, 21.6), flipped to the bottom, turned to 180 degrees
- moved C5 70.5 mm to (98.6, 21.6), turned to 0 degrees
- moved C73 70.2 mm to (38.2, 14.0), turned to 270 degrees
- moved R65 67.1 mm to (40.2, 14.0), flipped to the bottom, turned to 270 degrees
- moved R6 65.9 mm to (94.0, 16.0), flipped to the bottom, turned to 90 degrees
- moved C72 65.8 mm to (42.2, 14.0), flipped to the bottom, turned to 270 degrees
- moved C7 65.5 mm to (90.8, 13.2), flipped to the bottom, turned to 180 degrees
- moved R66 64.2 mm to (40.2, 11.0), flipped to the bottom, turned to 270 degrees
- moved C8 61.7 mm to (90.5, 19.2), flipped to the bottom, turned to 180 degrees
- moved IC3 60.3 mm to (91.0, 16.2), flipped to the bottom
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Connections:
- removed net 5V0@2: U$12.2, U$12.4
- removed net ACCELSA0: CPU.P$37, U2.P$7
- removed net ACCELSA1: CPU.P$38, IC$1.5
- removed net GND@3: U$12.25, U$12.39, U$12.9
- removed net GND@7: U$12.14, U$12.20, U$12.30, U$12.34, U$12.6
- removed net N$49: C93.1, CPU.P$48
- removed net N$51: C92.1, CPU.P$32
- removed net N$52: C73.1, IC10.2, R69.2
- removed net N$54: CPU.P$8, R44.1
- removed net N$71: C91.1, C95.1, CPU.P$13
- removed net N$78: C89.1, C90.1, CPU.P$1, CPU.P$19
- removed net N$80: C74.1, IC10.6, R72.2
- removed net STAGE1_DC_OFFSET: C19.1, C24.1, D3.1, D3.2, D4.1, D4.2, IC1.3, IC2.3, R25.2, R33.2
- removed net STAGE2_DC_OFFSET: C25.1, IC2.5, R32.2, R33.1, R9.1
- removed net STAGE3_DC_OFFSET: R67.2, R68.2, R69.1, R72.1
- removed net TEMP1: R4.1, R46.1, R48.1, R5.1
- removed net TEMP2: R4.2, R46.2, R48.2, R5.2
- removed net USER_0: CN1.3, CPU.P$52
- removed net USER_1: CN1.4, CPU.P$53
- removed net USER_2: CN1.5, CPU.P$2
- removed net USER_3: CN1.6, CPU.P$3
- new net DC_OFFSET: C19.1, C24.1, C25.1, C73.1, C74.1, D3.1, D3.2, D4.1, D4.2, IC1.3, IC10.3, IC10.5, IC2.3, IC2.5, R32.2, R68.2, R9.1
- new net N$10: D15.P$2, USB1.1
- net +3V3: now also C89.1, C90.1, C91.1, C92.1, C93.1, C94.1, C95.1, CPU.P$1, CPU.P$13, CPU.P$19, CPU.P$32, CPU.P$48, CPU.P$64, IC14.1, IC14.10, IC14.6, IC15.P$5, IC16.P$1, IC16.P$14, IC16.P$8, X4.1, X5.1; no longer CN1.1, IC$1.1, IC$1.10, IC$1.6, IC$2.P$5, J14.1, J6.1, U2.P$1, U2.P$14, U2.P$8
- net +4V: now also R4.1; no longer R25.1, R67.1
- net +5V: now also D15.P$1, IC17.6, J6.2, J6.4; no longer U$9.6, USB1.1
- net ACCELINT1: now also IC16.P$11, J6.33; no longer CPU.P$11, U2.P$11
- net ACCELINT2: now also IC16.P$9, J6.35; no longer CPU.P$24, U2.P$9
- net ACCELINT3: now also IC14.7, J6.37; no longer CPU.P$25, IC$1.7
- net AGND: now also D10.-, D12.-; no longer LED1.C, LED2.C, LED3.C, LED4.C, R32.1, R70.1, R76.1
- net BOOST: now also C48.2
- net CPU_BOOT0: now also J6.18; no longer U$12.18
- net CPU_JTCK-SWCLK: now also X4.7; no longer J14.4
- net CPU_JTDO-SWO: now also X4.2; no longer J14.8
- net CPU_JTMS-SWDIO: now also X4.5; no longer J14.3
- net CPU_NRST: now also J6.16, X4.8; no longer J14.5, U$12.16
- net CPU_SYS_JTDI: now also X4.6; no longer J14.6
- net CPU_SYS_JTRST: now also X4.4; no longer J14.7
- net GND: now also D1.-, D11.-, IC14.3, IC14.5, IC14.8, IC14.9, IC15.P$2, IC16.P$10, IC16.P$12, IC16.P$13, IC16.P$16, IC16.P$5, IC16.P$7, IC17.3, J6.14, J6.20, J6.25, J6.30, J6.34, J6.39, J6.6, J6.9, X2.P$2, X2.P$4, X4.3, X5.3; no longer C69.1, C70.1, CN1.2, D1.2, D1.4, D10.-, IC$1.3, IC$1.8, IC$1.9, IC$2.P$2, J14.2, J6.2, J7.2, J8.2, J9.2, U$9.3, U2.P$10, U2.P$12, U2.P$13, U2.P$16, U2.P$5
- net GPSPPS: now also CPU.P$14; no longer CPU.P$41
- net GPSRX: now also J6.8; no longer U$12.8
- net GPSTX: now also J6.10; no longer U$12.10
- net HV1EN: now also IC17.1; no longer U$9.1
- net HV1PWM: now also IC17.2; no longer U$9.2
- net HV2EN: now also IC17.8; no longer U$9.8
- net HV2PWM: now also IC17.4; no longer U$9.4
- net ID_SC: now also J6.28; no longer U$12.28
- net ID_SD: now also J6.27; no longer U$12.27
- net N$1: now also J3.5, R5.2; no longer D10.+, R44.2
- net N$12: now also IC10.2; no longer IC10.3
- net N$16: now also D13.2; no longer BAT46WH1.2
- net N$2: now also R4.2, R67.1; no longer C69.2, PSU.P$5, X2.P$1
- net N$20: now also D10.+; no longer LED1.A, LED3.A
- net N$21: now also R32.1, R67.2; no longer C94.1, CPU.P$64
- net N$28: now also D14.2; no longer BAT46WH2.2
- net N$3: now also D12.+; no longer LED2.A, LED4.A
- net N$30: now also D14.1; no longer BAT46WH2.1
- net N$34: now also IC17.5; no longer U$9.5
- net N$47: now also IC17.7; no longer U$9.7
- net N$59: now also IC10.6; no longer IC10.5
- net N$63: now also IC16.P$3; no longer U2.P$3
- net N$64: now also IC16.P$2; no longer U2.P$2
- net N$65: now also IC16.P$15; no longer U2.P$15
- net N$72: now also D1.+; no longer D1.1
- net N$73: now also D11.+; no longer D1.3
- net N$75: now also D13.1; no longer BAT46WH1.1
- net N$79: now also X2.P$3; no longer X3.P$1
- net N$8: now also J4.5, R25.2; no longer C70.2, PSU.P$6, X2.P$2
- net N$81: now also X2.P$1; no longer X3.P$2
- net PI_FLAG0: now also J6.7; no longer U$12.7
- net PI_FLAG1: now also J6.12; no longer U$12.12
- net PI_FLAG2: now also J6.15; no longer U$12.15
- net PSU_BOOT0: now also J6.13, PSU.P$60; no longer U$12.13
- net PSU_JTCK-SWCLK: now also X5.7; no longer J6.4
- net PSU_JTDO-SWO: now also X5.2; no longer J6.8
- net PSU_JTMS-SWDIO: now also X5.5; no longer J6.3
- net PSU_NRST: now also J6.11, X5.8; no longer J6.5, U$12.11
- net PSU_SYS_JTDI: now also X5.6; no longer J6.6
- net PSU_SYS_JTRST: now also X5.4; no longer J6.7
- net SCL0: now also IC14.2, IC15.P$6, IC16.P$4, J6.5; no longer IC$1.2, IC$2.P$6, U$12.5, U2.P$4
- net SDA0: now also IC14.4, IC15.P$1, IC16.P$6, J6.3; no longer IC$1.4, IC$2.P$1, U$12.3, U2.P$6
- net SLOWAOUT: now also CPU.P$23, R5.1; no longer CPU.P$15, J3.5, R70.2
- net SLOWBOUT: now also CPU.P$26, R25.1; no longer CPU.P$16, J4.5, R76.2
- net SPI_CE0: now also J6.24; no longer U$12.24
- net SPI_CE1: now also J6.26; no longer U$12.26
- net SPI_CLK: now also J6.23; no longer U$12.23
- net SPI_MISO: now also J6.21; no longer U$12.21
- net SPI_MOSI: now also CPU.P$57, J6.19; no longer CPU.P$23, U$12.19
- net STRIGAOUT: now also CPU.P$29; no longer CPU.P$43, J8.1
- net STRIGBOUT: now also CPU.P$17; no longer CPU.P$44, J9.1
- net SW: now also C48.1
- net TRIGOUT: now also CPU.P$15; no longer CPU.P$42, J7.1
Routing:
- net CASE: track 0.00 -> 793.6 mm, vias 0 -> 34
- net GND: track 664.9 -> 141.2 mm, vias 29 -> 62
- net AGND: track 278.8 -> 44.9 mm, vias 14 -> 24
- net STRIGB: track 229.3 -> 15.8 mm, vias 1 -> 3
- net GPSPPS: track 187.4 -> 27.6 mm, vias 5 -> 2
- net SPI_MISO: track 240.7 -> 87.9 mm, vias 4 -> 3
- net DC_OFFSET: track 0.00 -> 148.2 mm, vias 0 -> 11
- net SLOWBOUT: track 174.3 -> 27.1 mm, vias 4 -> 2
- net +5V: track 241.3 -> 99.5 mm, vias 16 -> 4
- net SDA0: track 185.8 -> 57.3 mm, vias 7 -> 4
- net GND@7: track 108.4 -> 0.00 mm, vias 5 -> 0
- net PSU_NRST: track 132.8 -> 25.2 mm, vias 6 -> 2
- net +3V3: track 491.5 -> 386.5 mm, vias 17 -> 19
- net HV2EN: track 122.1 -> 20.8 mm
- net CPU_SYS_JTDI: track 104.2 -> 3.86 mm, vias 0 -> 1
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- added copper zone on layer 1, net AGND
- added copper zone on layer 15, net AGND
- added copper zone on layer 16, net AGND
- added copper zone on layer 2, net AGND
- added copper zone on layer 1, net GND
- added copper zone on layer 15, net GND
- added copper zone on layer 16, net GND
- added copper zone on layer 2, net GND
Other:
- board size 120 x 159.8 mm -> 119 x 159.3 mm
- board text added: "Cosmic Pi V2 Main Board May '18 JD NB"
